File: pcb/Lucas11 GeometryPad.kicad_pcb (KiCad board)
At the start: 2 copper layers, 90.5 x 59.5 mm, 10 parts, among them J1 Conn_01x04_MountingPin, SW1 SW_Push, SW2 SW_Push, SW3 SW_Push, SW4 SW_Push, SW5 SW_Push, U1 XIAO-RP2040-DIP

Commit message: Break
Connections:
- SW2 pad 1: unconnected-(SW2-Pad1) -> GND
Routing:
- net Net-(U1-GPIO2/SCK): track 10.4 -> 129.6 mm
- net GND: track 117.5 -> 149.0 mm
- net Net-(U1-GPIO3/MOSI): track 23.8 -> 32.0 mm
- net Net-(J1-Pin_4): track 139.5 -> 145.0 mm
- net Net-(U1-GPIO28/ADC2/A2): track 116.5 -> 120.3 mm
- net Net-(J1-Pin_1): track 117.2 -> 119.7 mm
