File: pcb/Lucas11 GeometryPad.kicad_pcb (KiCad board)
At the start: 2 copper layers, 90.5 x 59.5 mm, 10 parts, among them J1 Conn_01x04_MountingPin, SW1 SW_Push, SW2 SW_Push, SW3 SW_Push, SW4 SW_Push, SW5 SW_Push, U1 XIAO-RP2040-DIP

Commit message: Fix some wireing
Routing:
- net Net-(U1-GPIO28/ADC2/A2): track 68.3 -> 74.4 mm
- net Net-(U1-GPIO3/MOSI): track 32.0 -> 37.2 mm
- net Net-(U1-GPIO4/MISO): track 65.9 -> 70.7 mm
- net Net-(J1-Pin_4): track 158.7 -> 154.5 mm
- net +5V: track 24.4 -> 27.2 mm
- net GND: track 185.8 -> 188.5 mm

Commit message: a
Connections:
- D1 pad 4: +5V -> VCC
- D2 pad 1: unconnected-(D2-DOUT-Pad1) -> Net-(D1-DIN)
- D2 pad 4: +5V -> VCC
- J1 pad 2: Net-(J1-Pin_2) -> VCC
- U1 pad 12: Net-(J1-Pin_2) -> VCC
- U1 pad 7: Net-(D1-DIN) -> unconnected-(U1-GPIO0/TX-Pad7)
Routing:
- net VCC: track 0.00 -> 227.8 mm
- net Net-(J1-Pin_2): track 199.3 -> 0.00 mm
- net GND: track 188.5 -> 135.9 mm
- net Net-(D1-DIN): track 45.4 -> 4.90 mm
- net +5V: track 27.2 -> 0.00 mm
- net Net-(D1-DOUT): track 8.32 -> 11.3 mm
