File: pcb/_autosave-Lucas11 GeometryPad.kicad_sch (KiCad schematic)
At the start: 9 parts, among them J1 Conn_01x04_MountingPin, SW1 SW_Push, SW2 SW_Push, SW3 SW_Push, SW4 SW_Push, SW5 SW_Push, U1 XIAO-RP2040-DIP

Commit message: Break
Changed lines of the file:
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@@
 		(pin "1"
-		)
-		(pin "MP"
 		)
 		(instances
