File: pcb/Lucas11 GeometryPad.kicad_sch (KiCad schematic)
At the start: 9 parts, among them J1 Conn_01x04_MountingPin, SW1 SW_Push, SW2 SW_Push, SW3 SW_Push, SW4 SW_Push, SW5 SW_Push, U1 XIAO-RP2040-DIP

Commit message: a
Connections:
- net +5V: no longer D1.4 (VDD), D2.4 (VDD)
- net VCC: now reaches J1.2 (Pin_2), U1.12 (3V3)
- net VCC: now also D1.4 (VDD), D2.4 (VDD)
- net at D1.3 (DIN): now also D2.1 (DOUT); no longer U1.7 (GPIO0/TX)
